File: Wiring Diagram/Wiring Diagram.kicad_sch (KiCad schematic)
At the start: 25 parts, among them J1 Raspberry Pi 4B, J10 Shovel Limit Switch, J2 Front Camera, J3 Back Camera, J4 ON Switch, J5 ON Switch, J6 E-Stop, J7 Solenoid Valve, J8 Right Steering Limit Switch, J9 Left Steering Limit Switch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

Commit message: Updated Wiring Diagram (with Wire Colours)
Connections:
- net +24V: now also U3. (VOUT); no longer U3.2 (FB), U3.4 (VOUT)
- net GND: now also U3. (VOUT); no longer J7. (IN-), U3.3 (GND)
- net at J1.13 (GPIO27): no longer U3.6 (EN)
- net at J1.19 (MOSI0/GPIO10): now also J8. (GND)
- net at J1.21 (MISO0/GPIO9): now also J9. (GND); no longer SW4.A (B)
- net at J1.23 (SCLK0/GPIO11): now also J10. (GND)
- net at J1.24 (~{CE0}/GPIO8): no longer SW4.B
- net at J1.26 (~{CE1}/GPIO7): now also U1.11 (EnB); no longer J10. (GND)
- net at J1.29 (GCLK1/GPIO5): now also U1.10 (IN3); no longer J9. (GND)
- net at J1.31 (GCLK2/GPIO6): now also U1.12 (IN4); no longer J8. (GND)
- net at J1.32 (PWM0/GPIO12): now also SW4.B; no longer J7. (IN-)
- net at J1.33 (PWM1/GPIO13): now also SW4.A (B); no longer J7. (IN-)
- net at U1.13 (OUT3): now also J7. (-)
- net at U1.14 (OUT4): now also J7. (-)
- removed net +12V: J4. (-), J7. (IN-), U3.1 (VIN)
- new net: J4. (-), U3. (VOUT)
Other:
- note added: "Black - USB Green - 24 AWG Blue - 12 AWG Red - 8 AWG"
